Commit message: proper camera position

File: dobot_magician/urdf/dobot_with_camera.urdf.xacro (robot description, xacro)
@@ -151,5 +151,5 @@
     <parent link="gripper_servo"/>
     <child link="camera_link"/>
-    <origin xyz="0.0 -0.0555 0.02" rpy="0 0 0"/>
+    <origin xyz="-0.0355 0.0 0.02" rpy="0 0 1.5708"/>
 </joint>
 </robot>
